File: Smart_fan_circuit/Smart_fan_circuit.kicad_sch (KiCad schematic)
At the start: 10 parts

Commit message: started working on BMS v1.101
Parts:
- removed Q? (x3): 2N2222A, digikey-footprints:TO-18-3, symbol dk_Transistors-Bipolar-BJT-Single:2N2222A
- added Q1, Q2, Q3, Q4: 2N2907A, symbol dk_Transistors-Bipolar-BJT-Single:2N2907A
- added Q6, Q7, Q8: 2N2222A, symbol dk_Transistors-Bipolar-BJT-Single:2N2222A
- added R1, R2, R3, R4, R5, R6, R7, R8: 2k, symbol Device:R
- added R10, R11, R12, R9: 10k, symbol Device:R
- C1: renamed from C?; value (none) -> 10uf, 20v
- C2: renamed from C?; value (none) -> 100nf
- J1: renamed from J?; value (none) -> 22-23-2021; footprint (none) -> digikey-footprints:PinHeader_1x2_P2.54mm_Drill1.02mm
- J2: renamed from J?; value (none) -> B5B-XH-A_LF__SN_; footprint (none) -> digikey-footprints:PinHeader_1x5_P2.5mm_Drill1.1mm
- Q5: renamed from Q?; footprint digikey-footprints:TO-18-3 -> (none)
- gave numbers to parts that had none: 2
Connections:
- net GND: now reaches Q5.1 (E)
- net GND: now also C1.2, C2.2, J1.1, J2.1, MOD1.1 (GND), U1.1 (GND), Q6.1 (E), Q7.1 (E), Q8.1 (E), R10.1, R11.1, R12.1, R9.1
- net at Q5.2 (B): now also R5.2, R9.2
- net IN1: now reaches Q5.3 (C)
- net IN1: now also R1.1
- net TX: now reaches MOD1.2 (TXO)
- net TX: now also R8.1
- net GPIO 2: now reaches MOD1.3 (GPIO2)
- net GPIO 2: now also R7.1
- net 3.3v: now reaches MOD1.4 (CHPD)
- net 3.3v: now also C2.1, MOD1.8 (3V), U1.2 (VO)
- net GPIO 0: now reaches MOD1.5 (GPIO0)
- net GPIO 0: now also R6.1
- net RX: now reaches MOD1.7 (RXI)
- net RX: now also R5.1
- net OUT1: now reaches J2.2
- net OUT1: now also Q1.3 (C)
- net OUT2: now reaches J2.3
- net OUT2: now also Q2.3 (C)
- net OUT3: now reaches J2.4
- net OUT3: now also Q3.3 (C)
- net OUT4: now reaches J2.5
- net OUT4: now also Q4.3 (C)
- net 5v: now reaches C1.1
- net 5v: now also J1.2, U1.3 (VI), Q1.1 (E), Q2.1 (E), Q3.1 (E), Q4.1 (E)
- new net: Q6.2 (B), R10.2, R6.2
- new net: Q1.2 (B), R1.2
- new net: Q8.2 (B), R12.2, R8.2
- new net: Q2.2 (B), R2.2
- new net: Q3.2 (B), R3.2
- new net: Q7.2 (B), R11.2, R7.2
- new net: Q4.2 (B), R4.2
- new net IN2: Q8.3 (C), R2.1
- new net IN3: Q6.3 (C), R3.1
- new net IN4: Q7.3 (C), R4.1
Other:
- moved on the sheet: C1, C2, J1, J2, MOD1, Q5, U1

Commit message: completed the fan circuit
Parts:
- U1: footprint Package_TO_SOT_SMD:SOT-223-3_TabPin2 -> (none)
Changed lines of the file:
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@@
     (property "Reference" "U1" (id 0) (at 58.42 21.59 0))
     (property "Value" "AMS1117-3.3" (id 1) (at 58.42 24.13 0))
-    (property "Footprint" "Package_TO_SOT_SMD:SOT-223-3_TabPin2" (id 2) (at 58.42 24.13 0)
+    (property "Footprint" "" (id 2) (at 58.42 24.13 0)
       (effects (font (size 1.27 1.27)) hide)
     )
@@
   (symbol_instances
     (path "/b17aea1f-56dd-4513-bc82-c4a6c326f278"
-      (reference "C1") (unit 1) (value "10uf, 20v") (footprint "")
+      (reference "C1") (unit 1) (value "10uf, 20v") (footprint "Capacitor_THT:CP_Radial_D5.0mm_P2.50mm")
     )
     (path "/892c2ce4-3701-4250-accf-fd778c33b016"
-      (reference "C2") (unit 1) (value "100nf") (footprint "")
+      (reference "C2") (unit 1) (value "100nf") (footprint "Capacitor_SMD:C_0603_1608Metric")
     )
     (path "/dd07efd4-24c4-483d-a118-ed58a9223c8c"
@@
     )
     (path "/1bea497f-a84d-41fd-8c04-7c9432823fdb"
-      (reference "R1") (unit 1) (value "2k") (footprint "Package_TO_SOT_SMD:SOT-23")
+      (reference "R1") (unit 1) (value "2k") (footprint "Resistor_SMD:R_0603_1608Metric")
     )
     (path "/f1b96db4-dc26-4eb6-94e5-34aad54dffd2"
-      (reference "R2") (unit 1) (value "2k") (footprint "Package_TO_SOT_SMD:SOT-23")
+      (reference "R2") (unit 1) (value "2k") (footprint "Resistor_SMD:R_0603_1608Metric")
     )
     (path "/54b4ec1b-13d4-4510-8abf-0b34fdfd6fa9"
-      (reference "R3") (unit 1) (value "2k") (footprint "Package_TO_SOT_SMD:SOT-23")
+      (reference "R3") (unit 1) (value "2k") (footprint "Resistor_SMD:R_0603_1608Metric")
     )
     (path "/c1ec2e1b-1582-4102-b131-0de181da6712"
-      (reference "R4") (unit 1) (value "2k") (footprint "Package_TO_SOT_SMD:SOT-23")
+      (reference "R4") (unit 1) (value "2k") (footprint "Resistor_SMD:R_0603_1608Metric")
     )
     (path "/58b94700-b19e-4d6b-86d1-5a2946640f08"
-      (reference "R5") (unit 1) (value "2k") (footprint "Package_TO_SOT_SMD:SOT-23")
+      (reference "R5") (unit 1) (value "2k") (footprint "Resistor_SMD:R_0603_1608Metric")
     )
     (path "/10ccd1f6-8ac0-41a6-beb0-93a566f4e739"
-      (reference "R6") (unit 1) (value "2k") (footprint "Package_TO_SOT_SMD:SOT-23")
+      (reference "R6") (unit 1) (value "2k") (footprint "Resistor_SMD:R_0603_1608Metric")
     )
     (path "/667abeaf-dd57-4992-b06e-3100b0f5c38a"
-      (reference "R7") (unit 1) (value "2k") (footprint "")
+      (reference "R7") (unit 1) (value "2k") (footprint "Resistor_SMD:R_0603_1608Metric")
     )
     (path "/5f7abf39-26f2-4536-b8f1-76a2d72c7a58"
-      (reference "R8") (unit 1) (value "2k") (footprint "")
+      (reference "R8") (unit 1) (value "2k") (footprint "Resistor_SMD:R_0603_1608Metric")
     )
     (path "/4db1f8a7-0ed9-499e-b9c7-c78238ae0fe3"
-      (reference "R9") (unit 1) (value "10k") (footprint "")
+      (reference "R9") (unit 1) (value "10k") (footprint "Resistor_SMD:R_0603_1608Metric")
     )
     (path "/38cbd0f1-9528-468e-aaf4-b0ba0d6b629e"
-      (reference "R10") (unit 1) (value "10k") (footprint "")
+      (reference "R10") (unit 1) (value "10k") (footprint "Resistor_SMD:R_0603_1608Metric")
     )
     (path "/b951ffdc-ca9f-46c3-aba2-5b22d1f3fc55"
-      (reference "R11") (unit 1) (value "10k") (footprint "")
+      (reference "R11") (unit 1) (value "10k") (footprint "Resistor_SMD:R_0603_1608Metric")
     )
     (path "/43452d5b-ba44-4473-b7ed-b0e4c7902559"
-      (reference "R12") (unit 1) (value "10k") (footprint "")
+      (reference "R12") (unit 1) (value "10k") (footprint "Resistor_SMD:R_0603_1608Metric")
     )
     (path "/ba8a5cbf-6c41-4bc4-a149-4dec895bdc0e"
-      (reference "U1") (unit 1) (value "AMS1117-3.3") (footprint "Package_TO_SOT_SMD:SOT-223-3_TabPin2")
-    )
-  )
+      (reference "U1") (unit 1) (value "AMS1117-3.3") (footprint "Package_TO_SOT_SMD:SOT-223")
+    )
+  )
